File: row_driver.brd (EAGLE design)
At the start: 27 parts, among them IC1 74HC138N, Q1 BC327, Q2 BC327, Q3 BC327, Q4 BC327, Q5 BC327, Q6 BC327, Q7 BC327, Q8 BC327

Commit message: row_driver: added GND and VCC
Connections:
- removed net N$6: IC1.6, JP2.4
- removed net N$7: IC1.4, IC1.5, JP2.5
- net GND: now also IC1.4, IC1.5, JP2.5
- net VCC: now also IC1.6, JP2.4
Changed lines of the file:
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@@
 <signal name="GND">
 <contactref element="IC1" pad="8"/>
+<contactref element="IC1" pad="5"/>
+<contactref element="IC1" pad="4"/>
+<contactref element="JP2" pad="5"/>
+<wire x1="1.27" y1="-22.86" x2="0" y2="-57.15" width="0" layer="19" extent="1-1"/>
+<wire x1="-1.27" y1="-22.86" x2="1.27" y2="-22.86" width="0" layer="19" extent="1-1"/>
+<wire x1="8.89" y1="-22.86" x2="1.27" y2="-22.86" width="0" layer="19" extent="1-1"/>
 </signal>
 <signal name="VCC">
 <contactref element="IC1" pad="16"/>
+<contactref element="JP2" pad="4"/>
+<contactref element="IC1" pad="6"/>
+<wire x1="3.81" y1="-22.86" x2="-2.54" y2="-57.15" width="0" layer="19" extent="1-1"/>
+<wire x1="-8.89" y1="-15.24" x2="3.81" y2="-22.86" width="0" layer="19" extent="1-1"/>
 </signal>
 <signal name="N$1">
@@
 <wire x1="-3.81" y1="-22.86" x2="-5.08" y2="-57.15" width="0" layer="19" extent="1-1"/>
 </signal>
-<signal name="N$6">
-<contactref element="JP2" pad="4"/>
-<contactref element="IC1" pad="6"/>
-<wire x1="3.81" y1="-22.86" x2="-2.54" y2="-57.15" width="0" layer="19" extent="1-1"/>
-</signal>
-<signal name="N$7">
-<contactref element="IC1" pad="5"/>
-<contactref element="IC1" pad="4"/>
-<contactref element="JP2" pad="5"/>
-<wire x1="1.27" y1="-22.86" x2="0" y2="-57.15" width="0" layer="19" extent="1-1"/>
-<wire x1="-1.27" y1="-22.86" x2="1.27" y2="-22.86" width="0" layer="19" extent="1-1"/>
-</signal>
 <signal name="N$8">
